Commit message: Fix robot_description asset references

File: src/robot_description/urdf/assets.urdf (robot description, URDF)
Before this commit: robot assets, 20 links, 19 joints
Links:
- link base_link: geometry collision mesh filename=package://robot_description/meshes/base_link.STL; visual mesh filename=package://robot_description/meshes/base_link.STL
- link right_ankle_1_3_cube_link: geometry collision mesh filename=package://robot_description/meshes/right_ankle_1_3_cube_lin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; visual mesh filename=package://robot_description/meshes/right_ankle_1_3_cube_lin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
- link right_ankle_1_3_link: geometry collision mesh filename=package://robot_description/meshes/right_ankle_1_3_link.STL; visual mesh filename=package://robot_description/meshes/right_ankle_1_3_link.STL
- link right_ankle_1_3_page_link: geometry collision mesh filename=package://robot_description/meshes/right_ankle_1_3_page_lin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; visual mesh filename=package://robot_description/meshes/right_ankle_1_3_page_lin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
- link right_ankle_2_3_cube_link: geometry collision mesh filename=package://robot_description/meshes/right_ankle_2_3_cube_lin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; visual mesh filename=package://robot_description/meshes/right_ankle_2_3_cube_lin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
- link right_ankle_2_3_link: geometry collision mesh filename=package://robot_description/meshes/right_ankle_2_3_link.STL; visual mesh filename=package://robot_description/meshes/right_ankle_2_3_link.STL
- link right_ankle_2_3_page_link: geometry collision mesh filename=package://robot_description/meshes/right_ankle_2_3_page_lin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; visual mesh filename=package://robot_description/meshes/right_ankle_2_3_page_lin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
- link right_ankle_3_3_cube_link: geometry collision mesh filename=package://robot_description/meshes/right_ankle_3_3_cube_lin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; visual mesh filename=package://robot_description/meshes/right_ankle_3_3_cube_lin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
- link right_ankle_3_3_link: geometry collision mesh filename=package://robot_description/meshes/right_ankle_3_3_link.STL; visual mesh filename=package://robot_description/meshes/right_ankle_3_3_link.STL
- link right_ankle_3_3_page_link: geometry collision mesh filename=package://robot_description/meshes/right_ankle_3_3_page_lin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; visual mesh filename=package://robot_description/meshes/right_ankle_3_3_page_lin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
- link right_ankle_axle_link: geometry collision mesh filename=package://robot_description/meshes/right_ankle_axle_link.STL; visual mesh filename=package://robot_description/meshes/right_ankle_axle_link.STL
- link right_ankle_cube_link: geometry collision mesh filename=package://robot_description/meshes/right_ankle_cube_link.STL; visual mesh filename=package://robot_description/meshes/right_ankle_cube_link.STL
- link right_foot_link: geometry collision mesh filename=package://robot_description/meshes/right_foot_link.STL; visual mesh filename=package://robot_description/meshes/right_foot_link.STL
- link right_hip_cube_link: geometry collision mesh filename=package://robot_description/meshes/right_hip_cube_link.STL; visual mesh filename=package://robot_description/meshes/right_hip_cube_link.STL
- link right_hip_pitch_engine_link: geometry collision mesh filename=package://robot_description/meshes/right_hip_pitch_engine_l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; visual mesh filename=package://robot_description/meshes/right_hip_pitch_engine_l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
- link right_hip_roll_link: geometry collision mesh filename=package://robot_description/meshes/right_hip_roll_link.STL; visual mesh filename=package://robot_description/meshes/right_hip_roll_link.STL
- link right_hip_yaw_engine_link: geometry collision mesh filename=package://robot_description/meshes/right_hip_yaw_engine_lin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; visual mesh filename=package://robot_description/meshes/right_hip_yaw_engine_lin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
- link right_shin_link: geometry collision mesh filename=package://robot_description/meshes/right_shin_link.STL; visual mesh filename=package://robot_description/meshes/right_shin_link.STL
- link right_thigh_link: geometry collision mesh filename=package://robot_description/meshes/right_thigh_link.STL; visual mesh filename=package://robot_description/meshes/right_thigh_link.STL
- link right_toe_link: geometry collision mesh filename=package://robot_description/meshes/right_toe_link.STL; visual mesh filename=package://robot_description/meshes/right_toe_link.STL
