Commit message: Update robot_description assets

File: src/robot_description/urdf/assets.urdf (robot description, URDF)
Before this commit: robot assets, 20 links, 19 joints
Links:
- removed link right_ankle_1_3_cube_link
- removed link right_ankle_1_3_link
- removed link right_ankle_1_3_page_link
- removed link right_ankle_2_3_cube_link
- removed link right_ankle_2_3_link
- removed link right_ankle_2_3_page_link
- removed link right_ankle_3_3_cube_link
- removed link right_ankle_3_3_link
- removed link right_ankle_3_3_page_link
- added link left_ankle_axle_link, mass 0.00188539443116976; collision mesh filename=package://robot_description/meshes/left_ankle_axle_link.STL; visual mesh filename=package://robot_description/meshes/left_ankle_axle_link.STL
- added link left_ankle_cube_link, mass 0.000189328304341637; collision mesh filename=package://robot_description/meshes/left_ankle_cube_link.STL; visual mesh filename=package://robot_description/meshes/left_ankle_cube_link.STL
- added link left_arm_link, mass 0.0463841814445341; collision mesh filename=package://robot_description/meshes/left_arm_link.STL; visual mesh filename=package://robot_description/meshes/left_arm_link.STL
- added link left_branch_link, mass 0.013497890740739; collision mesh filename=package://robot_description/meshes/left_branch_link.STL; visual mesh filename=package://robot_description/meshes/left_branch_link.STL
- added link left_foot_link, mass 0.138474623900114; collision mesh filename=package://robot_description/meshes/left_foot_link.STL; visual mesh filename=package://robot_description/meshes/left_foot_link.STL
- added link left_forearm_link, mass 0.0295290267369982; collision mesh filename=package://robot_description/meshes/left_forearm_link.STL; visual mesh filename=package://robot_description/meshes/left_forearm_link.STL
- added link left_hand_link, mass 0.00350581330345173; collision mesh filename=package://robot_description/meshes/left_hand_link.STL; visual mesh filename=package://robot_description/meshes/left_hand_link.STL
- added link left_hip_cube_link, mass 0.000245876972106249; collision mesh filename=package://robot_description/meshes/left_hip_cube_link.STL; visual mesh filename=package://robot_description/meshes/left_hip_cube_link.STL
- added link left_hip_pitch_engine_link, mass 0.0068093; collision mesh filename=package://robot_description/meshes/left_hip_pitch_engine_li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; visual mesh filename=package://robot_description/meshes/left_hip_pitch_engine_li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
- added link left_hip_roll_link, mass 0.00374844887826709; collision mesh filename=package://robot_description/meshes/left_hip_roll_link.STL; visual mesh filename=package://robot_description/meshes/left_hip_roll_link.STL
- added link left_hip_yaw_engine_link, mass 0.0074512; collision mesh filename=package://robot_description/meshes/left_hip_yaw_engine_link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; visual mesh filename=package://robot_description/meshes/left_hip_yaw_engine_link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
- added link left_shin_link, mass 0.34781395968867; collision mesh filename=package://robot_description/meshes/left_shin_link.STL; visual mesh filename=package://robot_description/meshes/left_shin_link.STL
- added link left_shoulder_link, mass 5.463E-05; collision mesh filename=package://robot_description/meshes/left_shoulder_link.STL; visual mesh filename=package://robot_description/meshes/left_shoulder_link.STL
- added link left_spine_003_link, mass 0.019257; collision mesh filename=package://robot_description/meshes/left_spine_003_link.STL; visual mesh filename=package://robot_description/meshes/left_spine_003_link.STL
- added link left_spine_004_ground_link, mass 0.0371077097805639; collision mesh filename=package://robot_description/meshes/left_spine_004_ground_li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; visual mesh filename=package://robot_description/meshes/left_spine_004_ground_li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
- added link left_spine_004_link, mass 0.00196590214384826; collision mesh filename=package://robot_description/meshes/left_spine_004_link.STL; visual mesh filename=package://robot_description/meshes/left_spine_004_link.STL
- added link left_thigh_link, mass 0.65016; collision mesh filename=package://robot_description/meshes/left_thigh_link.STL; visual mesh filename=package://robot_description/meshes/left_thigh_link.STL
- added link left_toe_link, mass 0.0528822247684934; collision mesh filename=package://robot_description/meshes/left_toe_link.STL; visual mesh filename=package://robot_description/meshes/left_toe_link.STL
- added link left_wrist_cube_link, mass 0.00188539503253632; collision mesh filename=package://robot_description/meshes/left_wrist_cube_link.STL; visual mesh filename=package://robot_description/meshes/left_wrist_cube_link.STL
- added link left_wrist_link, mass 0.000189328304341632; collision mesh filename=package://robot_description/meshes/left_wrist_link.STL; visual mesh filename=package://robot_description/meshes/left_wrist_link.STL
- added link neck_axle_link, mass 0.00172774344297369; collision mesh filename=package://robot_description/meshes/neck_axle_link.STL; visual mesh filename=package://robot_description/meshes/neck_axle_link.STL
- added link neck_cube_link, mass 0.0140124948869863; collision mesh filename=package://robot_description/meshes/neck_cube_link.STL; visual mesh filename=package://robot_description/meshes/neck_cube_link.STL
- added link right_arm_link, mass 0.0463841814445341; collision mesh filename=package://robot_description/meshes/right_arm_link.STL; visual mesh filename=package://robot_description/meshes/right_arm_link.STL
- added link right_branch_link, mass 0.013497890740739; collision mesh filename=package://robot_description/meshes/right_branch_link.STL; visual mesh filename=package://robot_description/meshes/right_branch_link.STL
- added link right_forearm_link, mass 0.0295290267369982; collision mesh filename=package://robot_description/meshes/right_forearm_link.STL; visual mesh filename=package://robot_description/meshes/right_forearm_link.STL
- added link right_hand_link, mass 0.00350581330345173; collision mesh filename=package://robot_description/meshes/right_hand_link.STL; visual mesh filename=package://robot_description/meshes/right_hand_link.STL
- added link right_shoulder_link, mass 5.463E-05; collision mesh filename=package://robot_description/meshes/right_shoulder_link.STL; visual mesh filename=package://robot_description/meshes/right_shoulder_link.STL
- added link right_spine_003_link, mass 0.019257; collision mesh filename=package://robot_description/meshes/right_spine_003_link.STL; visual mesh filename=package://robot_description/meshes/right_spine_003_link.STL
- added link right_spine_004_ground_link, mass 0.0371077097805639; collision mesh filename=package://robot_description/meshes/right_spine_004_ground_l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; visual mesh filename=package://robot_description/meshes/right_spine_004_ground_l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
- added link right_spine_004_link, mass 0.00196590214384826; collision mesh filename=package://robot_description/meshes/right_spine_004_link.STL; visual mesh filename=package://robot_description/meshes/right_spine_004_link.STL
- added link right_wrist_cube_link, mass 0.00188539503253632; collision mesh filename=package://robot_description/meshes/right_wrist_cube_link.STL; visual mesh filename=package://robot_description/meshes/right_wrist_cube_link.STL
- added link right_wrist_link, mass 0.000189328304341632; collision mesh filename=package://robot_description/meshes/right_wrist_link.STL; visual mesh filename=package://robot_description/meshes/right_wrist_link.STL
- added link spine_001_axle_link, mass 0.00172774341614448; collision mesh filename=package://robot_description/meshes/spine_001_axle_link.STL; visual mesh filename=package://robot_description/meshes/spine_001_axle_link.STL
- added link spine_001_cube_link, mass 0.00018933; collision mesh filename=package://robot_description/meshes/spine_001_cube_link.STL; visual mesh filename=package://robot_description/meshes/spine_001_cube_link.STL
- added link spine_001_link, mass 0.0320197009924435; collision mesh filename=package://robot_description/meshes/spine_001_link.STL; visual mesh filename=package://robot_description/meshes/spine_001_link.STL
- added link spine_002_axle_link, mass 0.000510082145710689; collision mesh filename=package://robot_description/meshes/spine_002_axle_link.STL; visual mesh filename=package://robot_description/meshes/spine_002_axle_link.STL
- added link spine_002_cube_link, mass 0.000189328304341632; collision mesh filename=package://robot_description/meshes/spine_002_cube_link.STL; visual mesh filename=package://robot_description/meshes/spine_002_cube_link.STL
- added link spine_002_link, mass 0.030952; collision mesh filename=package://robot_description/meshes/spine_002_link.STL; visual mesh filename=package://robot_description/meshes/spine_002_link.STL
- added link spine_003_axle_link, mass 0.000510082296418304; collision mesh filename=package://robot_description/meshes/spine_003_axle_link.STL; visual mesh filename=package://robot_description/meshes/spine_003_axle_link.STL
- added link spine_003_cube_link, mass 0.03220902930632; collision mesh filename=package://robot_description/meshes/spine_003_cube_link.STL; visual mesh filename=package://robot_description/meshes/spine_003_cube_link.STL
- added link spine_003_link, mass 0.000510082123516246; collision mesh filename=package://robot_description/meshes/spine_003_link.STL; visual mesh filename=package://robot_description/meshes/spine_003_link.STL
- added link spine_004_axle_link, mass 0.000189328304341632; collision mesh filename=package://robot_description/meshes/spine_004_axle_link.STL; visual mesh filename=package://robot_description/meshes/spine_004_axle_link.STL
- added link spine_004_cube_link, mass 0.0123462395112595; collision mesh filename=package://robot_description/meshes/spine_004_cube_link.STL; visual mesh filename=package://robot_description/meshes/spine_004_cube_link.STL
- added link spine_004_link, mass 0.000189328304341631; collision mesh filename=package://robot_description/meshes/spine_004_link.STL; visual mesh filename=package://robot_description/meshes/spine_004_link.STL
- link base_link: mass 0.557304827590303 -> 0.57845
- link right_ankle_axle_link: mass 0.0018856554715005 -> 0.00188539443116976
- link right_ankle_cube_link: mass 0.000189328304341634 -> 0.000189328304341637
- link right_foot_link: mass 0.17435588732169 -> 0.138474623900114
- link right_hip_cube_link: mass 0.000245876972106248 -> 0.000245876972106249
- link right_hip_pitch_engine_link: mass 0.00784384827917925 -> 0.0068093
- link right_hip_roll_link: mass 0.00398432706561057 -> 0.00374844887826709
- link right_hip_yaw_engine_link: mass 0.00721229273746498 -> 0.0074512
- link right_shin_link: mass 0.364323955321575 -> 0.34781395968867
- link right_thigh_link: mass 0.807844023825405 -> 0.65016
- link right_toe_link: mass 0.0528820880759984 -> 0.0528822247684934
Joints:
- removed joint right_ankle_1_3_cube_joint
- removed joint right_ankle_1_3_joint
- removed joint right_ankle_1_3_page_joint
- removed joint right_ankle_2_3_cube_joint
- removed joint right_ankle_2_3_joint
- removed joint right_ankle_2_3_page_joint
- removed joint right_ankle_3_3_cube_joint
- removed joint right_ankle_3_3_joint
- removed joint right_ankle_3_3_page_joint
- added joint base_joint: type revolute, parent base_link, child spine_001_axle_link, origin xyz=0 0.087689 0.002418 rpy=0.2618 0.00052789 0.00014145, axis 0 1 0, limit lower=-3.14 upper=3.14 effort=100 velocity=1
- added joint left_ankle_axle_joint: type revolute, parent left_ankle_cube_link, child left_ankle_axle_link, origin xyz=0.02567 -0.88669 0.0080049 rpy=0 0 -0, axis -1 0 0, limit lower=-3.14 upper=3.14 effort=100 velocity=1
- added joint left_ankle_cube_joint: type revolute, parent left_shin_link, child left_ankle_cube_link, origin xyz=-0.025667 0.42982 0.0115 rpy=0 0 -0, axis -0 0 1, limit lower=-3.14 upper=3.14 effort=100 velocity=1
- added joint left_branch_link: type fixed, parent spine_002_link, child left_branch_link, origin xyz=0.077264 0.10221 0.0074994 rpy=3.161e-05 0.11474 0.0074894, axis -0 0 0, limit lower=-3.14 upper=3.14 effort=100 velocity=1
- added joint left_elbow_joint: type revolute, parent left_arm_link, child left_forearm_link, origin xyz=0.045652 -0.19823 0.027394 rpy=-0.13165 -0.17347 0.024955, axis 1 0 0, limit lower=-3.14 upper=3.14 effort=100 velocity=1
- added joint left_foot_joint: type revolute, parent left_ankle_axle_link, child left_foot_link, origin xyz=-0 -0.01475 0 rpy=0 0 -0, axis -0 -1 0, limit lower=-3.14 upper=3.14 effort=100 velocity=1
- added joint left_forearm_joint: type revolute, parent left_forearm_link, child left_wrist_link, origin xyz=0.00015 -0.24101 0.11283 rpy=0.44847 0 -3.14159, axis -0 0 -1, limit lower=-3.14 upper=3.14 effort=100 velocity=1
- added joint left_hand_cube_joint: type revolute, parent left_wrist_cube_link, child left_hand_link, origin xyz=-0 0 0 rpy=0 0 -0, axis -0 -1 0, limit lower=-3.14 upper=3.14 effort=100 velocity=1
- added joint left_hip_cube_joint: type revolute, parent left_hip_roll_link, child left_hip_cube_link, origin xyz=-0 0 0 rpy=0 0 -0, axis -0 0 1, limit lower=-3.14 upper=3.14 effort=100 velocity=1
- added joint left_hip_pitch_engine_joint: type revolute, parent base_link, child left_hip_pitch_engine_link, origin xyz=0.084333 2.4595e-05 0 rpy=0 0 -0, axis -0 0 1, limit lower=-3.14 upper=3.14 effort=100 velocity=1
- added joint left_hip_roll_joint: type revolute, parent base_link, child left_hip_roll_link, origin xyz=0.084333 2.4595e-05 0 rpy=0 0 -0, axis 1 0 0, limit lower=-3.14 upper=3.14 effort=100 velocity=1
- added joint left_hip_yaw_engine_joint: type revolute, parent base_link, child left_hip_yaw_engine_link, origin xyz=0.084333 2.4595e-05 0 rpy=0 0 -0, axis -0 1 0, limit lower=-3.14 upper=3.14 effort=100 velocity=1
- added joint left_knee_joint: type revolute, parent left_thigh_link, child left_shin_link, origin xyz=0.025667 -0.42982 -0.0115 rpy=0 0 -0, axis -1 0 0, limit lower=-3.14 upper=3.14 effort=100 velocity=1
- added joint left_shoulder_joint: type revolute, parent left_shoulder_link, child left_arm_link, origin xyz=-0 0 0 rpy=0 0 -0, axis -0.00085941 -0.087156 0.99619, limit lower=-3.14 upper=3.14 effort=100 velocity=1
- added joint left_spine_002_joint: type revolute, parent left_branch_link, child left_spine_003_link, origin xyz=-0 0 0 rpy=0 0 -0, axis -0.00027429 -1 0, limit lower=-3.14 upper=3.14 effort=100 velocity=1
- added joint left_spine_003_joint: type revolute, parent left_spine_003_link, child left_spine_004_ground_link, origin xyz=0.0041074 0.072996 -0.046784 rpy=0 1.4837 -0.00027429, axis 1 0 0, limit lower=-3.14 upper=3.14 effort=100 velocity=1
- added joint left_spine_004_ground_joint: type revolute, parent left_spine_004_ground_link, child left_spine_004_link, origin xyz=-0.043245 0.042061 0.051578 rpy=-0.39852 -1.5704 0.66032, axis -1 -0.00044361 -0.0009015, limit lower=-3.14 upper=3.14 effort=100 velocity=1
- added joint left_spine_004_joint: type revolute, parent left_spine_004_link, child left_shoulder_link, origin xyz=-0 0 0 rpy=0 0 -0, axis -0.00085941 -0.087156 0.99619, limit lower=-3.14 upper=3.14 effort=100 velocity=1
- added joint left_thigh_joint: type revolute, parent left_hip_cube_link, child left_thigh_link, origin xyz=-0 0 0 rpy=0 0 -0, axis -0 1 0, limit lower=-3.14 upper=3.14 effort=100 velocity=1
- added joint left_toe_joint: type revolute, parent left_foot_link, child left_toe_link, origin xyz=-0.00050001 -0.064606 0.10561 rpy=0 0 -0, axis -1 0 0, limit lower=-3.14 upper=3.14 effort=100 velocity=1
- added joint left_wrist_cube_joint: type revolute, parent left_wrist_link, child left_wrist_cube_link, origin xyz=-0 0 0 rpy=0 0 -0, axis -1 0 0, limit lower=-3.14 upper=3.14 effort=100 velocity=1
- added joint neck_axle_joint: type revolute, parent neck_axle_link, child neck_cube_link, origin xyz=0.0018322 0.030834 0.0026322 rpy=0.087233 0.22756 -0.039767, axis 0.00014644 -1 0, limit lower=-3.14 upper=3.14 effort=100 velocity=1
- added joint right_branch_link: type fixed, parent spine_002_link, child right_branch_link, origin xyz=-0.077264 0.10221 0.0074994 rpy=3.161E-05 -0.11474 -0.0074894, axis 0 0 0, limit lower=-3.14 upper=3.14 effort=100 velocity=1
- added joint right_elbow_joint: type revolute, parent right_arm_link, child right_forearm_link, origin xyz=-0.045652 -0.19823 0.027394 rpy=-0.13165 0.17347 -0.024955, axis -1 0 0, limit lower=-3.14 upper=3.14 effort=100 velocity=1
- added joint right_forearm_joint: type revolute, parent right_forearm_link, child right_wrist_link, origin xyz=-0.00015 -0.24101 0.11283 rpy=0.44847 0 -3.1416, axis 0 0 -1, limit lower=-3.14 upper=3.14 effort=100 velocity=1
- added joint right_hand_cube_joint: type revolute, parent right_wrist_cube_link, child right_hand_link, origin xyz=0 0 0 rpy=0 0 0, axis 0 -1 0, limit lower=-3.14 upper=3.14 effort=100 velocity=1
- added joint right_shoulder_joint: type revolute, parent right_shoulder_link, child right_arm_link, origin xyz=0 0 0 rpy=0 0 0, axis 0.00085941 -0.087156 0.99619, limit lower=-3.14 upper=3.14 effort=100 velocity=1
- added joint right_spine_002_joint: type revolute, parent right_branch_link, child right_spine_003_link, origin xyz=0 0 0 rpy=0 0 0, axis 0.00027429 -1 0, limit lower=-3.14 upper=3.14 effort=100 velocity=1
- added joint right_spine_003_joint: type revolute, parent right_spine_003_link, child right_spine_004_ground_link, origin xyz=-0.0041074 0.072996 -0.046784 rpy=0 -1.4837 0.00027429, axis -1 0 0, limit lower=-3.14 upper=3.14 effort=100 velocity=1
- added joint right_spine_004_ground_joint: type revolute, parent right_spine_004_ground_link, child right_spine_004_link, origin xyz=0.043245 0.042061 0.051578 rpy=-0.39852 1.5704 -0.66032, axis 1 -0.00044361 -0.0009015, limit lower=-3.14 upper=3.14 effort=100 velocity=1
- added joint right_spine_004_joint: type revolute, parent right_spine_004_link, child right_shoulder_link, origin xyz=0 0 0 rpy=0 0 0, axis 0.00085941 -0.087156 0.99619, limit lower=-3.14 upper=3.14 effort=100 velocity=1
- added joint right_wrist_cube_joint: type revolute, parent right_wrist_link, child right_wrist_cube_link, origin xyz=0 0 0 rpy=0 0 0, axis 1 0 0, limit lower=-3.14 upper=3.14 effort=100 velocity=1
- added joint spine_001_axle_joint: type revolute, parent spine_001_axle_link, child spine_001_cube_link, origin xyz=0 0.011 0 rpy=-0.34415 0.17488 0, axis -1 0 0, limit lower=-3.14 upper=3.14 effort=100 velocity=1
- added joint spine_001_cube_joint: type revolute, parent spine_001_cube_link, child spine_001_link, origin xyz=0 0 0 rpy=0 0 0, axis 0 0 1, limit lower=-3.14 upper=3.14 effort=100 velocity=1
- added joint spine_001_joint: type revolute, parent spine_001_link, child spine_002_axle_link, origin xyz=0.0067007 0.1124 0 rpy=3.1034E-05 -0.16453 -0.059733, axis -0.00018692 1 0, limit lower=-3.14 upper=3.14 effort=100 velocity=1
- added joint spine_002_axle_join: type revolute, parent spine_002_axle_link, child spine_002_cube_link, origin xyz=0 0.011 0 rpy=-0.1744 0.028305 0.002522, axis 1 -0.0023701 0, limit lower=-3.14 upper=3.14 effort=100 velocity=1
- added joint spine_002_cube_join: type revolute, parent spine_002_cube_link, child spine_002_link, origin xyz=0 0 0 rpy=0 0 0, axis 0 0 -1, limit lower=-3.14 upper=3.14 effort=100 velocity=1
- added joint spine_002_joint: type revolute, parent spine_002_link, child spine_003_axle_link, origin xyz=0.00080644 0.1118 0 rpy=0 -0.02747 -0.0074866, axis 0.00027325 -1 0, limit lower=-3.14 upper=3.14 effort=100 velocity=1
- added joint spine_003_axle_joint: type revolute, parent spine_003_axle_link, child spine_003_cube_link, origin xyz=0 0.011 0 rpy=0.1861 0.25101 0.068889, axis 0.99773 -0.067369 0, limit lower=-3.14 upper=3.14 effort=100 velocity=1
- added joint spine_003_cube_joint: type revolute, parent spine_003_cube_link, child spine_003_link, origin xyz=0.0025012 0.11227 0 rpy=4.9543E-05 -0.2591 -0.022468, axis -0.00018692 1 0, limit lower=-3.14 upper=3.14 effort=100 velocity=1
- added joint spine_003_joint: type revolute, parent spine_003_link, child spine_004_axle_link, origin xyz=0 0.011 0 rpy=0.25994 0.21059 0.018747, axis -0.99982 0.018761 0, limit lower=-3.14 upper=3.14 effort=100 velocity=1
- added joint spine_004_axle_joint: type revolute, parent spine_004_axle_link, child spine_004_cube_link, origin xyz=0 0 0 rpy=0 0 0, axis 0 0 1, limit lower=-3.14 upper=3.14 effort=100 velocity=1
- added joint spine_004_cube_joint: type revolute, parent spine_004_cube_link, child spine_004_link, origin xyz=-0.0047469 0.12971 0 rpy=-0.018441 -0.43543 0.080276, axis 0 0 1, limit lower=-3.14 upper=3.14 effort=100 velocity=1
- added joint spine_004_joint: type revolute, parent spine_004_link, child neck_axle_link, origin xyz=0 0 0 rpy=0 0 0, axis 0.99824 -0.059317 0, limit lower=-3.14 upper=3.14 effort=100 velocity=1
- joint right_ankle_axle_joint: origin xyz=0 0 0 rpy=0 0 0 -> xyz=-0.02567 -0.88669 0.0080049 rpy=0 0 0
- joint right_ankle_cube_joint: origin xyz=0.00500000000000023 -0.451000010144081 0.0244999999999944 rpy=0 0 0 -> xyz=0.025667 0.42982 0.0115 rpy=0 0 0
- joint right_foot_joint: origin xyz=0 -0.019999989834798 0 rpy=0 0 0 -> xyz=0 -0.01475 0 rpy=0 0 0
- joint right_hip_pitch_engine_joint: origin xyz=-0.084333 2.46E-05 0 rpy=0 0 0 -> xyz=-0.084333 2.4595E-05 0 rpy=0 0 0
- joint right_hip_roll_joint: axis 1 0 0 -> -1 0 0; origin xyz=-0.084333 2.46E-05 0 rpy=0 0 0 -> xyz=-0.084333 2.4595E-05 0 rpy=0 0 0
- joint right_hip_yaw_engine_joint: origin xyz=-0.084333 2.46E-05 0 rpy=0 0 0 -> xyz=-0.084333 2.4595E-05 0 rpy=0 0 0
- joint right_knee_joint: axis -1 0 0 -> 1 0 0; origin xyz=-0.0324938548812839 -0.429595785329822 -0.011499999999998 rpy=0 0 0 -> xyz=-0.025667 -0.42982 -0.0115 rpy=0 0 0
- joint right_toe_joint: origin xyz=0 -0.0758129417355203 0.0950624781069581 rpy=0 0 0 -> xyz=0.00050001 -0.064606 0.10561 rpy=0 0 0
