Commit message: fix:robot and web_stream

File: src/robot_description/urdf/jiyuan.urdf (robot description, URDF)
Before this commit: robot jiyuan_bilateral_bilateral, 56 links, 55 joints
Links:
- link base_link: geometry collision mesh filename=package://jiyuan/meshes/base_link.STL; visual mesh filename=package://jiyuan/meshes/base_link.STL
- link left_ankle_axle_link: geometry collision mesh filename=package://jiyuan/meshes/left_ankle_axle_link.STL; visual mesh filename=package://jiyuan/meshes/left_ankle_axle_link.STL
- link left_ankle_cube_link: geometry collision mesh filename=package://jiyuan/meshes/left_ankle_cube_link.STL; visual mesh filename=package://jiyuan/meshes/left_ankle_cube_link.STL
- link left_arm_link: geometry collision mesh filename=package://jiyuan/meshes/left_arm_link.STL; visual mesh filename=package://jiyuan/meshes/left_arm_link.STL
- link left_branch_link: geometry collision mesh filename=package://jiyuan/meshes/left_branch_link.STL; visual mesh filename=package://jiyuan/meshes/left_branch_link.STL
- link left_foot_link: geometry collision mesh filename=package://jiyuan/meshes/left_foot_link.STL; visual mesh filename=package://jiyuan/meshes/left_foot_link.STL
- link left_forearm_link: geometry collision mesh filename=package://jiyuan/meshes/left_forearm_link.STL; visual mesh filename=package://jiyuan/meshes/left_forearm_link.STL
- link left_hand_link: geometry collision mesh filename=package://jiyuan/meshes/left_hand_link.STL; visual mesh filename=package://jiyuan/meshes/left_hand_link.STL
- link left_hip_cube_link: geometry collision mesh filename=package://jiyuan/meshes/left_hip_cube_link.STL; visual mesh filename=package://jiyuan/meshes/left_hip_cube_link.STL
- link left_hip_pitch_engine_link: geometry collision mesh filename=package://jiyuan/meshes/left_hip_pitch_engine_link.STL; visual mesh filename=package://jiyuan/meshes/left_hip_pitch_engine_link.STL
- link left_hip_roll_link: geometry collision mesh filename=package://jiyuan/meshes/left_hip_roll_link.STL; visual mesh filename=package://jiyuan/meshes/left_hip_roll_link.STL
- link left_hip_yaw_engine_link: geometry collision mesh filename=package://jiyuan/meshes/left_hip_yaw_engine_link.STL; visual mesh filename=package://jiyuan/meshes/left_hip_yaw_engine_link.STL
- link left_shin_link: geometry collision mesh filename=package://jiyuan/meshes/left_shin_link.STL; visual mesh filename=package://jiyuan/meshes/left_shin_link.STL
- link left_shoulder_link: geometry collision mesh filename=package://jiyuan/meshes/left_shoulder_link.STL; visual mesh filename=package://jiyuan/meshes/left_shoulder_link.STL
- link left_spine_003_link: geometry collision mesh filename=package://jiyuan/meshes/left_spine_003_link.STL; visual mesh filename=package://jiyuan/meshes/left_spine_003_link.STL
- link left_spine_004_ground_link: geometry collision mesh filename=package://jiyuan/meshes/left_spine_004_ground_link.STL; visual mesh filename=package://jiyuan/meshes/left_spine_004_ground_link.STL
- link left_spine_004_link: geometry collision mesh filename=package://jiyuan/meshes/left_spine_004_link.STL; visual mesh filename=package://jiyuan/meshes/left_spine_004_link.STL
- link left_thigh_link: geometry collision mesh filename=package://jiyuan/meshes/left_thigh_link.STL; visual mesh filename=package://jiyuan/meshes/left_thigh_link.STL
- link left_toe_link: geometry collision mesh filename=package://jiyuan/meshes/left_toe_link.STL; visual mesh filename=package://jiyuan/meshes/left_toe_link.STL
- link left_wrist_cube_link: geometry collision mesh filename=package://jiyuan/meshes/left_wrist_cube_link.STL; visual mesh filename=package://jiyuan/meshes/left_wrist_cube_link.STL
- link left_wrist_link: geometry collision mesh filename=package://jiyuan/meshes/left_wrist_link.STL; visual mesh filename=package://jiyuan/meshes/left_wrist_link.STL
- link neck_axle_link: geometry collision mesh filename=package://jiyuan/meshes/neck_axle_link.STL; visual mesh filename=package://jiyuan/meshes/neck_axle_link.STL
- link neck_cube_link: geometry collision mesh filename=package://jiyuan/meshes/neck_cube_link.STL; visual mesh filename=package://jiyuan/meshes/neck_cube_link.STL
- link neck_link: geometry collision mesh filename=package://jiyuan/meshes/neck_link.STL; visual mesh filename=package://jiyuan/meshes/neck_link.STL
- link right_ankle_axle_link: geometry collision mesh filename=package://jiyuan/meshes/right_ankle_axle_link.STL; visual mesh filename=package://jiyuan/meshes/right_ankle_axle_link.STL
- link right_ankle_cube_link: geometry collision mesh filename=package://jiyuan/meshes/right_ankle_cube_link.STL; visual mesh filename=package://jiyuan/meshes/right_ankle_cube_link.STL
- link right_arm_link: geometry collision mesh filename=package://jiyuan/meshes/right_arm_link.STL; visual mesh filename=package://jiyuan/meshes/right_arm_link.STL
- link right_branch_link: geometry collision mesh filename=package://jiyuan/meshes/right_branch_link.STL; visual mesh filename=package://jiyuan/meshes/right_branch_link.STL
- link right_foot_link: geometry collision mesh filename=package://jiyuan/meshes/right_foot_link.STL; visual mesh filename=package://jiyuan/meshes/right_foot_link.STL
- link right_forearm_link: geometry collision mesh filename=package://jiyuan/meshes/right_forearm_link.STL; visual mesh filename=package://jiyuan/meshes/right_forearm_link.STL
- link right_hand_link: geometry collision mesh filename=package://jiyuan/meshes/right_hand_link.STL; visual mesh filename=package://jiyuan/meshes/right_hand_link.STL
- link right_hip_cube_link: geometry collision mesh filename=package://jiyuan/meshes/right_hip_cube_link.STL; visual mesh filename=package://jiyuan/meshes/right_hip_cube_link.STL
- link right_hip_pitch_engine_link: geometry collision mesh filename=package://jiyuan/meshes/right_hip_pitch_engine_link.STL; visual mesh filename=package://jiyuan/meshes/right_hip_pitch_engine_link.STL
- link right_hip_roll_link: geometry collision mesh filename=package://jiyuan/meshes/right_hip_roll_link.STL; visual mesh filename=package://jiyuan/meshes/right_hip_roll_link.STL
- link right_hip_yaw_engine_link: geometry collision mesh filename=package://jiyuan/meshes/right_hip_yaw_engine_link.STL; visual mesh filename=package://jiyuan/meshes/right_hip_yaw_engine_link.STL
- link right_shin_link: geometry collision mesh filename=package://jiyuan/meshes/right_shin_link.STL; visual mesh filename=package://jiyuan/meshes/right_shin_link.STL
- link right_shoulder_link: geometry collision mesh filename=package://jiyuan/meshes/right_shoulder_link.STL; visual mesh filename=package://jiyuan/meshes/right_shoulder_link.STL
- link right_spine_003_link: geometry collision mesh filename=package://jiyuan/meshes/right_spine_003_link.STL; visual mesh filename=package://jiyuan/meshes/right_spine_003_link.STL
- link right_spine_004_ground_link: geometry collision mesh filename=package://jiyuan/meshes/right_spine_004_ground_link.STL; visual mesh filename=package://jiyuan/meshes/right_spine_004_ground_link.STL
- link right_spine_004_link: geometry collision mesh filename=package://jiyuan/meshes/right_spine_004_link.STL; visual mesh filename=package://jiyuan/meshes/right_spine_004_link.STL
- link right_thigh_link: geometry collision mesh filename=package://jiyuan/meshes/right_thigh_link.STL; visual mesh filename=package://jiyuan/meshes/right_thigh_link.STL
- link right_toe_link: geometry collision mesh filename=package://jiyuan/meshes/right_toe_link.STL; visual mesh filename=package://jiyuan/meshes/right_toe_link.STL
- link right_wrist_cube_link: geometry collision mesh filename=package://jiyuan/meshes/right_wrist_cube_link.STL; visual mesh filename=package://jiyuan/meshes/right_wrist_cube_link.STL
- link right_wrist_link: geometry collision mesh filename=package://jiyuan/meshes/right_wrist_link.STL; visual mesh filename=package://jiyuan/meshes/right_wrist_link.STL
- link spine_001_axle_link: geometry collision mesh filename=package://jiyuan/meshes/spine_001_axle_link.STL; visual mesh filename=package://jiyuan/meshes/spine_001_axle_link.STL
- link spine_001_cube_link: geometry collision mesh filename=package://jiyuan/meshes/spine_001_cube_link.STL; visual mesh filename=package://jiyuan/meshes/spine_001_cube_link.STL
- link spine_001_link: geometry collision mesh filename=package://jiyuan/meshes/spine_001_link.STL; visual mesh filename=package://jiyuan/meshes/spine_001_link.STL
- link spine_002_axle_link: geometry collision mesh filename=package://jiyuan/meshes/spine_002_axle_link.STL; visual mesh filename=package://jiyuan/meshes/spine_002_axle_link.STL
- link spine_002_cube_link: geometry collision mesh filename=package://jiyuan/meshes/spine_002_cube_link.STL; visual mesh filename=package://jiyuan/meshes/spine_002_cube_link.STL
- link spine_002_link: geometry collision mesh filename=package://jiyuan/meshes/spine_002_link.STL; visual mesh filename=package://jiyuan/meshes/spine_002_link.STL
- link spine_003_axle_link: geometry collision mesh filename=package://jiyuan/meshes/spine_003_axle_link.STL; visual mesh filename=package://jiyuan/meshes/spine_003_axle_link.STL
- link spine_003_cube_link: geometry collision mesh filename=package://jiyuan/meshes/spine_003_cube_link.STL; visual mesh filename=package://jiyuan/meshes/spine_003_cube_link.STL
- link spine_003_link: geometry collision mesh filename=package://jiyuan/meshes/spine_003_link.STL; visual mesh filename=package://jiyuan/meshes/spine_003_link.STL
- link spine_004_axle_link: geometry collision mesh filename=package://jiyuan/meshes/spine_004_axle_link.STL; visual mesh filename=package://jiyuan/meshes/spine_004_axle_link.STL
- link spine_004_cube_link: geometry collision mesh filename=package://jiyuan/meshes/spine_004_cube_link.STL; visual mesh filename=package://jiyuan/meshes/spine_004_cube_link.STL
- link spine_004_link: geometry collision mesh filename=package://jiyuan/meshes/spine_004_link.STL; visual mesh filename=package://jiyuan/meshes/spine_004_link.STL
