Commit message: fix:robot and web_stream

File: src/robot_description/urdf/jiyuan_bilateral.urdf (robot description, URDF)
Before this commit: robot jiyuan_bilateral_bilateral, 56 links, 55 joints
Links:
- removed link neck_link
- link base_link: mass 0.578447340656943 -> 0.57845; geometry collision mesh filename=package://jiyuan/meshes/base_link.STL; visual mesh filename=package://jiyuan/meshes/base_link.STL
- link left_ankle_axle_link: geometry collision mesh filename=package://jiyuan/meshes/left_ankle_axle_link.STL; visual mesh filename=package://jiyuan/meshes/left_ankle_axle_link.STL
- link left_ankle_cube_link: mass 0.000189328304341638 -> 0.000189328304341637; geometry collision mesh filename=package://jiyuan/meshes/left_ankle_cube_link.STL; visual mesh filename=package://jiyuan/meshes/left_ankle_cube_link.STL
- link left_arm_link: geometry collision mesh filename=package://jiyuan/meshes/left_arm_link.STL; visual mesh filename=package://jiyuan/meshes/left_arm_link.STL
- link left_branch_link: geometry collision mesh filename=package://jiyuan/meshes/left_branch_link.STL; visual mesh filename=package://jiyuan/meshes/left_branch_link.STL
- link left_foot_link: mass 0.138474623900111 -> 0.138474623900114; geometry collision mesh filename=package://jiyuan/meshes/left_foot_link.STL; visual mesh filename=package://jiyuan/meshes/left_foot_link.STL
- link left_forearm_link: geometry collision mesh filename=package://jiyuan/meshes/left_forearm_link.STL; visual mesh filename=package://jiyuan/meshes/left_forearm_link.STL
- link left_hand_link: geometry collision mesh filename=package://jiyuan/meshes/left_hand_link.STL; visual mesh filename=package://jiyuan/meshes/left_hand_link.STL
- link left_hip_cube_link: geometry collision mesh filename=package://jiyuan/meshes/left_hip_cube_link.STL; visual mesh filename=package://jiyuan/meshes/left_hip_cube_link.STL
- link left_hip_pitch_engine_link: mass 0.00680931690813817 -> 0.0068093; geometry collision mesh filename=package://jiyuan/meshes/left_hip_pitch_engine_link.STL; visual mesh filename=package://jiyuan/meshes/left_hip_pitch_engine_link.STL
- link left_hip_roll_link: geometry collision mesh filename=package://jiyuan/meshes/left_hip_roll_link.STL; visual mesh filename=package://jiyuan/meshes/left_hip_roll_link.STL
- link left_hip_yaw_engine_link: mass 0.00745115887807254 -> 0.0074512; geometry collision mesh filename=package://jiyuan/meshes/left_hip_yaw_engine_link.STL; visual mesh filename=package://jiyuan/meshes/left_hip_yaw_engine_link.STL
- link left_shin_link: mass 0.347813967537165 -> 0.34781395968867; geometry collision mesh filename=package://jiyuan/meshes/left_shin_link.STL; visual mesh filename=package://jiyuan/meshes/left_shin_link.STL
- link left_shoulder_link: mass 5.46299456939302E-05 -> 5.463E-05; geometry collision mesh filename=package://jiyuan/meshes/left_shoulder_link.STL; visual mesh filename=package://jiyuan/meshes/left_shoulder_link.STL
- link left_spine_003_link: mass 0.0192570395361066 -> 0.019257; geometry collision mesh filename=package://jiyuan/meshes/left_spine_003_link.STL; visual mesh filename=package://jiyuan/meshes/left_spine_003_link.STL
- link left_spine_004_ground_link: geometry collision mesh filename=package://jiyuan/meshes/left_spine_004_ground_link.STL; visual mesh filename=package://jiyuan/meshes/left_spine_004_ground_link.STL
- link left_spine_004_link: mass 0.00196590214384828 -> 0.00196590214384826; geometry collision mesh filename=package://jiyuan/meshes/left_spine_004_link.STL; visual mesh filename=package://jiyuan/meshes/left_spine_004_link.STL
- link left_thigh_link: mass 0.651256730970666 -> 0.65016; geometry collision mesh filename=package://jiyuan/meshes/left_thigh_link.STL; visual mesh filename=package://jiyuan/meshes/left_thigh_link.STL
- link left_toe_link: mass 0.0528822247684903 -> 0.0528822247684934; geometry collision mesh filename=package://jiyuan/meshes/left_toe_link.STL; visual mesh filename=package://jiyuan/meshes/left_toe_link.STL
- link left_wrist_cube_link: geometry collision mesh filename=package://jiyuan/meshes/left_wrist_cube_link.STL; visual mesh filename=package://jiyuan/meshes/left_wrist_cube_link.STL
- link left_wrist_link: geometry collision mesh filename=package://jiyuan/meshes/left_wrist_link.STL; visual mesh filename=package://jiyuan/meshes/left_wrist_link.STL
- link neck_axle_link: mass 0.000189328304341631 -> 0.00172774344297369; geometry collision mesh filename=package://jiyuan/meshes/neck_axle_link.STL; visual mesh filename=package://jiyuan/meshes/neck_axle_link.STL
- link neck_cube_link: mass 0.00172774344297369 -> 0.0140124948869863; geometry collision mesh filename=package://jiyuan/meshes/neck_cube_link.STL; visual mesh filename=package://jiyuan/meshes/neck_cube_link.STL
- link right_ankle_axle_link: geometry collision mesh filename=package://jiyuan/meshes/right_ankle_axle_link.STL; visual mesh filename=package://jiyuan/meshes/right_ankle_axle_link.STL
- link right_ankle_cube_link: mass 0.000189328304341638 -> 0.000189328304341637; geometry collision mesh filename=package://jiyuan/meshes/right_ankle_cube_link.STL; visual mesh filename=package://jiyuan/meshes/right_ankle_cube_link.STL
- link right_arm_link: geometry collision mesh filename=package://jiyuan/meshes/right_arm_link.STL; visual mesh filename=package://jiyuan/meshes/right_arm_link.STL
- link right_branch_link: geometry collision mesh filename=package://jiyuan/meshes/right_branch_link.STL; visual mesh filename=package://jiyuan/meshes/right_branch_link.STL
- link right_foot_link: mass 0.138474623900111 -> 0.138474623900114; geometry collision mesh filename=package://jiyuan/meshes/right_foot_link.STL; visual mesh filename=package://jiyuan/meshes/right_foot_link.STL
- link right_forearm_link: geometry collision mesh filename=package://jiyuan/meshes/right_forearm_link.STL; visual mesh filename=package://jiyuan/meshes/right_forearm_link.STL
- link right_hand_link: geometry collision mesh filename=package://jiyuan/meshes/right_hand_link.STL; visual mesh filename=package://jiyuan/meshes/right_hand_link.STL
- link right_hip_cube_link: geometry collision mesh filename=package://jiyuan/meshes/right_hip_cube_link.STL; visual mesh filename=package://jiyuan/meshes/right_hip_cube_link.STL
- link right_hip_pitch_engine_link: mass 0.00680931690813817 -> 0.0068093; geometry collision mesh filename=package://jiyuan/meshes/right_hip_pitch_engine_link.STL; visual mesh filename=package://jiyuan/meshes/right_hip_pitch_engine_link.STL
- link right_hip_roll_link: geometry collision mesh filename=package://jiyuan/meshes/right_hip_roll_link.STL; visual mesh filename=package://jiyuan/meshes/right_hip_roll_link.STL
- link right_hip_yaw_engine_link: mass 0.00745115887807254 -> 0.0074512; geometry collision mesh filename=package://jiyuan/meshes/right_hip_yaw_engine_link.STL; visual mesh filename=package://jiyuan/meshes/right_hip_yaw_engine_link.STL
- link right_shin_link: mass 0.347813967537165 -> 0.34781395968867; geometry collision mesh filename=package://jiyuan/meshes/right_shin_link.STL; visual mesh filename=package://jiyuan/meshes/right_shin_link.STL
- link right_shoulder_link: mass 5.46299456939302E-05 -> 5.463E-05; geometry collision mesh filename=package://jiyuan/meshes/right_shoulder_link.STL; visual mesh filename=package://jiyuan/meshes/right_shoulder_link.STL
- link right_spine_003_link: mass 0.0192570395361066 -> 0.019257; geometry collision mesh filename=package://jiyuan/meshes/right_spine_003_link.STL; visual mesh filename=package://jiyuan/meshes/right_spine_003_link.STL
- link right_spine_004_ground_link: geometry collision mesh filename=package://jiyuan/meshes/right_spine_004_ground_link.STL; visual mesh filename=package://jiyuan/meshes/right_spine_004_ground_link.STL
- link right_spine_004_link: mass 0.00196590214384828 -> 0.00196590214384826; geometry collision mesh filename=package://jiyuan/meshes/right_spine_004_link.STL; visual mesh filename=package://jiyuan/meshes/right_spine_004_link.STL
- link right_thigh_link: mass 0.651256730970666 -> 0.65016; geometry collision mesh filename=package://jiyuan/meshes/right_thigh_link.STL; visual mesh filename=package://jiyuan/meshes/right_thigh_link.STL
- link right_toe_link: mass 0.0528822247684903 -> 0.0528822247684934; geometry collision mesh filename=package://jiyuan/meshes/right_toe_link.STL; visual mesh filename=package://jiyuan/meshes/right_toe_link.STL
- link right_wrist_cube_link: geometry collision mesh filename=package://jiyuan/meshes/right_wrist_cube_link.STL; visual mesh filename=package://jiyuan/meshes/right_wrist_cube_link.STL
- link right_wrist_link: geometry collision mesh filename=package://jiyuan/meshes/right_wrist_link.STL; visual mesh filename=package://jiyuan/meshes/right_wrist_link.STL
- link spine_001_axle_link: geometry collision mesh filename=package://jiyuan/meshes/spine_001_axle_link.STL; visual mesh filename=package://jiyuan/meshes/spine_001_axle_link.STL
- link spine_001_cube_link: mass 0.000189328304341632 -> 0.00018933; geometry collision mesh filename=package://jiyuan/meshes/spine_001_cube_link.STL; visual mesh filename=package://jiyuan/meshes/spine_001_cube_link.STL
- link spine_001_link: geometry collision mesh filename=package://jiyuan/meshes/spine_001_link.STL; visual mesh filename=package://jiyuan/meshes/spine_001_link.STL
- link spine_002_axle_link: geometry collision mesh filename=package://jiyuan/meshes/spine_002_axle_link.STL; visual mesh filename=package://jiyuan/meshes/spine_002_axle_link.STL
- link spine_002_cube_link: geometry collision mesh filename=package://jiyuan/meshes/spine_002_cube_link.STL; visual mesh filename=package://jiyuan/meshes/spine_002_cube_link.STL
- link spine_002_link: mass 0.0309518546203202 -> 0.030952; geometry collision mesh filename=package://jiyuan/meshes/spine_002_link.STL; visual mesh filename=package://jiyuan/meshes/spine_002_link.STL
- link spine_003_axle_link: geometry collision mesh filename=package://jiyuan/meshes/spine_003_axle_link.STL; visual mesh filename=package://jiyuan/meshes/spine_003_axle_link.STL
- link spine_003_cube_link: mass 0.000189328304341632 -> 0.03220902930632; geometry collision mesh filename=package://jiyuan/meshes/spine_003_cube_link.STL; visual mesh filename=package://jiyuan/meshes/spine_003_cube_link.STL
- link spine_003_link: mass 0.0320197010019784 -> 0.000510082123516246; geometry collision mesh filename=package://jiyuan/meshes/spine_003_link.STL; visual mesh filename=package://jiyuan/meshes/spine_003_link.STL
- link spine_004_axle_link: mass 0.000510082123516246 -> 0.000189328304341632; geometry collision mesh filename=package://jiyuan/meshes/spine_004_axle_link.STL; visual mesh filename=package://jiyuan/meshes/spine_004_axle_link.STL
- link spine_004_cube_link: mass 0.000189328304341632 -> 0.0123462395112595; geometry collision mesh filename=package://jiyuan/meshes/spine_004_cube_link.STL; visual mesh filename=package://jiyuan/meshes/spine_004_cube_link.STL
- link spine_004_link: mass 0.0123462395112595 -> 0.000189328304341631; geometry collision mesh filename=package://jiyuan/meshes/spine_004_link.STL; visual mesh filename=package://jiyuan/meshes/spine_004_link.STL
Joints:
- removed joint left_spine_004_ground_joint
- removed joint neck_joint
- removed joint right_spine_004_ground_joint
- joint left_ankle_axle_joint: origin xyz=0.02567 -0.886686 0.00800489 rpy=0 0 -0 -> xyz=0.02567 -0.88669 0.0080049 rpy=0 0 -0
- joint left_ankle_cube_joint: origin xyz=-0.0256668 0.429825 0.0115 rpy=0 0 -0 -> xyz=-0.025667 0.42982 0.0115 rpy=0 0 -0
- joint left_branch_link: origin xyz=0.0772641 0.10221 0.00749937 rpy=3.16096e-05 0.114737 0.00748937 -> xyz=0.077264 0.10221 0.0074994 rpy=3.161e-05 0.11474 0.0074894
- joint left_elbow_joint: origin xyz=0.0456519 -0.198226 0.0273941 rpy=-0.131652 -0.173467 0.024955 -> xyz=0.045652 -0.19823 0.027394 rpy=-0.13165 -0.17347 0.024955
- joint left_forearm_joint: origin xyz=0.00015 -0.241007 0.112833 rpy=0.448472 0 3.14159 -> xyz=0.00015 -0.24101 0.11283 rpy=0.44847 0 -3.14159
- joint left_hip_pitch_engine_joint: origin xyz=0.0843332 2.45945e-05 0 rpy=0 0 -0 -> xyz=0.084333 2.4595e-05 0 rpy=0 0 -0
- joint left_hip_roll_joint: origin xyz=0.0843332 2.45945e-05 0 rpy=0 0 -0 -> xyz=0.084333 2.4595e-05 0 rpy=0 0 -0
- joint left_hip_yaw_engine_joint: origin xyz=0.0843332 2.45945e-05 0 rpy=0 0 -0 -> xyz=0.084333 2.4595e-05 0 rpy=0 0 -0
- joint left_knee_joint: origin xyz=0.0256668 -0.429825 -0.0115 rpy=0 0 -0 -> xyz=0.025667 -0.42982 -0.0115 rpy=0 0 -0
- joint left_shoulder_joint: axis -0.000859407 -0.0871558 0.996194 -> -0.00085941 -0.087156 0.99619
- joint left_spine_002_joint: axis -0.000274286 -1 0 -> -0.00027429 -1 0
- joint left_spine_003_joint: axis 1 0 0 -> -1 -0.00044361 -0.0009015; child left_spine_004_ground_link -> left_spine_004_link; origin xyz=0.00410736 0.0729963 -0.0467839 rpy=3.11428e-19 1.48365 -0.000274286 -> xyz=-0.043245 0.042061 0.051578 rpy=-0.39852 -1.5704 0.66032; parent left_spine_003_link -> left_spine_004_ground_link
- joint left_spine_004_joint: axis -0.000859407 -0.0871558 0.996194 -> -0.00085941 -0.087156 0.99619
- joint left_toe_joint: origin xyz=-0.0005 -0.0646056 0.105615 rpy=0 0 -0 -> xyz=-0.00050001 -0.064606 0.10561 rpy=0 0 -0
- joint neck_axle_joint: axis 0.97403 0.00014263 0.22641 -> 0.00014644 -1 0
- joint right_ankle_axle_joint: origin xyz=-0.0256700103430628 -0.886686499663044 0.00800489064197998 rpy=0 0 0 -> xyz=-0.02567 -0.88669 0.0080049 rpy=0 0 0
- joint right_ankle_cube_joint: origin xyz=0.025666845538777 0.429824594538245 0.0115000000000049 rpy=0 0 0 -> xyz=0.025667 0.42982 0.0115 rpy=0 0 0
- joint right_branch_link: origin xyz=-0.0772640532330563 0.102209980220283 0.00749936807653298 rpy=3.16095910023056E-05 -0.114736944872298 -0.00748936555497514 -> xyz=-0.077264 0.10221 0.0074994 rpy=3.161E-05 -0.11474 -0.0074894
- joint right_elbow_joint: origin xyz=-0.0456518822542674 -0.198226035200409 0.0273940850548131 rpy=-0.13165218489478 0.173467112582246 -0.0249549558994513 -> xyz=-0.045652 -0.19823 0.027394 rpy=-0.13165 0.17347 -0.024955
- joint right_foot_joint: origin xyz=0 -0.0147499860831098 0 rpy=0 0 0 -> xyz=0 -0.01475 0 rpy=0 0 0
- joint right_forearm_joint: origin xyz=-0.000150000010252893 -0.241006694344342 0.112832954897592 rpy=0.448472339283537 0 -3.14159265358979 -> xyz=-0.00015 -0.24101 0.11283 rpy=0.44847 0 -3.1416
- joint right_hip_pitch_engine_joint: origin xyz=-0.084333154461223 2.45945382447853E-05 0 rpy=0 0 0 -> xyz=-0.084333 2.4595E-05 0 rpy=0 0 0
- joint right_hip_roll_joint: origin xyz=-0.084333154461223 2.45945382447853E-05 0 rpy=0 0 0 -> xyz=-0.084333 2.4595E-05 0 rpy=0 0 0
- joint right_hip_yaw_engine_joint: origin xyz=-0.084333154461223 2.45945382447853E-05 0 rpy=0 0 0 -> xyz=-0.084333 2.4595E-05 0 rpy=0 0 0
- joint right_knee_joint: origin xyz=-0.025666845538777 -0.429824594538245 -0.0115000000000049 rpy=0 0 0 -> xyz=-0.025667 -0.42982 -0.0115 rpy=0 0 0
- joint right_shoulder_joint: axis 0.000859407421352749 -0.0871557532121165 0.996194326474967 -> 0.00085941 -0.087156 0.99619
- joint right_spine_002_joint: axis 0.000274286186586446 -0.999999962383543 0 -> 0.00027429 -1 0
- joint right_spine_003_joint: axis -1 0 0 -> 1 -0.00044361 -0.0009015; child right_spine_004_ground_link -> right_spine_004_link; origin xyz=-0.00410736211631267 0.072996321531915 -0.0467839448006484 rpy=0 -1.48365130116614 0.000274286189964258 -> xyz=0.043245 0.042061 0.051578 rpy=-0.39852 1.5704 -0.66032; parent right_spine_003_link -> right_spine_004_ground_link
- joint right_spine_004_joint: axis 0.000859407421352749 -0.0871557532121165 0.996194326474967 -> 0.00085941 -0.087156 0.99619
- joint right_toe_joint: origin xyz=0.000499999710812979 -0.0646056174661427 0.105614593490204 rpy=0 0 0 -> xyz=0.00050001 -0.064606 0.10561 rpy=0 0 0
- joint spine_001_axle_joint: origin xyz=0 0.011 0 rpy=-0.344154933334362 0.174881984566998 0 -> xyz=0 0.011 0 rpy=-0.34415 0.17488 0
- joint spine_001_joint: axis -0.000186916583478837 0.999999982531095 0 -> -0.00018692 1 0; origin xyz=0.00670068441639467 0.112400448523802 0 rpy=3.10340201864658E-05 -0.164530504019474 -0.0597333970241516 -> xyz=0.0067007 0.1124 0 rpy=3.1034E-05 -0.16453 -0.059733
- joint spine_002_axle_join: axis 0.99999719125963 -0.00237012085153487 0 -> 1 -0.0023701 0; origin xyz=0 0.0109999998078421 0 rpy=-0.17440079274189 0.0283053809155349 0.00252199483425913 -> xyz=0 0.011 0 rpy=-0.1744 0.028305 0.002522
- joint spine_002_joint: axis 0.000273253759191587 -0.999999962666191 0 -> 0.00027325 -1 0; origin xyz=0.000806435919506334 0.111797091469804 0 rpy=0 -0.0274704855817947 -0.00748662087643142 -> xyz=0.00080644 0.1118 0 rpy=0 -0.02747 -0.0074866
- joint spine_003_axle_joint: axis 0.997728143633419 -0.0673687717107211 0 -> 0.99773 -0.067369 0; origin xyz=0 0.0109999995893339 0 rpy=0.186095390069988 0.251012260294841 0.0688886558053852 -> xyz=0 0.011 0 rpy=0.1861 0.25101 0.068889
- joint spine_003_cube_joint: axis 0 0 1 -> -0.00018692 1 0; origin xyz=0 0 0 rpy=0 0 0 -> xyz=0.0025012 0.11227 0 rpy=4.9543E-05 -0.2591 -0.022468
- joint spine_003_joint: axis -0.000186916583478925 0.999999982531095 0 -> -0.99982 0.018761 0; origin xyz=0.00250119688024906 0.112272142645293 0 rpy=4.95430163599117E-05 -0.259096323257594 -0.0224676694074587 -> xyz=0 0.011 0 rpy=0.25994 0.21059 0.018747
- joint spine_004_axle_joint: axis -0.999824004673546 0.0187605884383361 0 -> 0 0 1; origin xyz=0 0.0109999998063652 0 rpy=0.259937971789517 0.210585098557286 0.0187470971171111 -> xyz=0 0 0 rpy=0 0 0
- joint spine_004_cube_joint: origin xyz=0 0 0 rpy=0 0 0 -> xyz=-0.0047469 0.12971 0 rpy=-0.018441 -0.43543 0.080276
- joint spine_004_joint: axis 0 0 1 -> 0.99824 -0.059317 0; origin xyz=-0.00474688798162995 0.129713172249461 0 rpy=-0.0184410969908424 -0.435431971027392 0.0802758501201312 -> xyz=0 0 0 rpy=0 0 0
